File: 2024-2025_Boards/LED_Board/LED_Board.kicad_sch (KiCad schematic)
At the start: 58 parts, among them J1 Conn_01x02_Socket, J10 22232031, J11 22232031, J12 22232031, J13 22232031, J14 22232031, J2 Conn_01x02_Socket, J3 Conn_ARM_JTAG_SWD_10, J4 Conn_01x03_Socket, J5 Conn_01x03_Socket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

Commit message: Replaced footprints and new power/can connector
Parts:
- removed D1, D2: MMBZ27VCLT1G, CMR_Voltage_Suppressor:SOT95P237X111-3N, symbol Voltage_Supressor:MMBZ27VCLT1G
- removed J1, J2: Conn_01x02_Socket, Connector_AMASS:AMASS_XT30PW-M_1x02_P2.50mm_Horizontal, symbol Connector:Conn_01x02_Socket
- removed J4, J5: Conn_01x03_Socket, Connector_JST:JST_PH_S3B-PH-SM4-TB_1x03-1MP_P2.00mm_Horizontal, symbol Connector:Conn_01x03_Socket
- removed J8: 54-00236, LED_Board_Schematic:TENSILITY_54-00236, symbol LED_Board_Schematic-eagle-import:M12-5P_54-00236
- removed U5, U6: CSD88537NDD8-M, LED_Board_Schematic:D8-M, symbol LED_Board_Schematic-eagle-import:CMR_CSD88537NDD8-M
- added D1, D2: MMBZ27VCLT1G, CMR_Voltage_Suppressor:SOT95P237X111-3N, symbol CMR_Voltage_Suppressor:MMBZ27VCLT1G
- added J1, J2: 3007W2PAT73A10X, CMR_Power_CAN_Connector:3007W2PAT73A10X, symbol CMR_Power_CAN_Connector:3007W2PAT73A10X
- added J8: 54-00236, CMR_LED_Array_Pins:TENSILITY_54-00236, symbol CMR_LED_Array_Pins:54-00236
- added U5, U6: CSD88537ND, CMR_N_Channel_Power_Mosfet:CSD88537ND8-M, symbol CMR_N_Channel_Power_Mosfet:CSD88537ND
- J10, J11, J12, J13, J14, J9: footprint CONN_A-6373-03A_MOL -> CMR_Fan_Pin_Header:CONN_A-6373-03A_MOL
Connections:
- net CAN_H: now also D1.2, J1.4, J2.4
- net CAN_L: now also D2.2, J1.2, J2.2
- net G1: now also TP4.1, U4.11 (PA3)
- net G2: now also TP5.1, U4.12 (PA4)
- net G3: now also TP6.1, U4.13 (PA5)
- net G4: now also TP7.1, U4.14 (PA6)
- net GND: now also D1.1, D2.1, J1.3, J1.N, J2.3, J2.N, U5.1 (S1), U5.3 (S2), U6.1 (S1), U6.3 (S2)
- net LED_1: now also J8.1, U5.7 (D1), U5.8 (D1); no longer TP4.1
- net LED_2: now also J8.2, U5.5 (D2), U5.6 (D2); no longer TP5.1
- net LED_3: now also J8.4, U6.7 (D1), U6.8 (D1); no longer TP6.1
- net LED_4: now also J8.5, U6.5 (D2), U6.6 (D2); no longer TP7.1
- net LED_Debug: now also U4.9 (PA1); no longer U4.11 (PA3)
- net V_IN: now also J1.P, J2.P, J8.3
- net at R10.2, R12.1: now also U6.4 (G2)
- net at R6.2, R8.1: now also U5.4 (G2)
- net at R11.1, R9.2: now also U6.2 (G1)
- net at R5.2, R7.1: now also U5.2 (G1)
- no-connect marks 39 -> 33
Other:
- moved on the sheet: C5, C6, C7, D3, D4, J3, J6, J7, R1, R2, R3, U3

Commit message: New connector and board layout progress
Parts:
- removed J2: 3007W2PAT73A10X, CMR_Power_CAN_Connector:3007W2PAT73A10X, symbol CMR_Power_CAN_Connector:3007W2PAT73A10X
- removed J8: 54-00236, CMR_LED_Array_Pins:TENSILITY_54-00236, symbol CMR_LED_Array_Pins:54-00236
- removed R4: 0, Resistor_SMD:R_0402_1005Metric, symbol Device:R
- removed U3: MCP2562-E-P, Package_DIP:DIP-8_W7.62mm, symbol Interface_CAN_LIN:MCP2562-E-P
- added J2: Conn_01x02_Socket, Connector_AMASS:AMASS_XT30PW-M_1x02_P2.50mm_Horizontal, symbol Connector:Conn_01x02_Socket
- added J3: Conn_01x03_Socket, Connector_JST:JST_PH_S3B-PH-SM4-TB_1x03-1MP_P2.00mm_Horizontal, symbol Connector:Conn_01x03_Socket
- added J7: 54-00236, CMR_LED_Array_Pins:TENSILITY_54-00236, symbol CMR_LED_Array_Pins:54-00236
- added U3: TCAN1057AEV-Q1, Package_SO:SOIC-8_3.9x4.9mm_P1.27mm, symbol moteus:TCAN1042HGVDRBRQ1
- C5, C6: value 100n -> 1u
- renumbered J3 to J4, J6 to J5, J7 to J6
Connections:
- net 3.3V: now also C6.1, U3.5 (VIO); no longer C5.1
- net 5V: now also C5.1, U3.3 (VCC); no longer C6.2
- net CAN_H: now also J1.5, J3.1 (Pin_1), U3.7 (CANH); no longer J1.4
- net CAN_L: now also J1.1, J3.2 (Pin_2), U3.6 (CANL); no longer J1.2
- net CAN_RX: now also U3.4 (RXD)
- net CAN_TX: now also U3.1 (TXD)
- net GND: now also C6.2, J1.2, J1.A2, J2.1 (Pin_1), J3.3 (Pin_3), U3.2 (GND), U3.8 (STB), U3.9 (PAD); no longer C6.1, J1.3, J1.N
- net LED_1: now also J7.1
- net LED_2: now also J7.2
- net LED_3: now also J7.4
- net LED_4: now also J7.5
- net SWO: now also U4.40 (PB3)
- net V_IN: now also J1.A1, J2.2 (Pin_2); no longer J1.P
- net V_Fuse: now reaches C1.1, F1.2, F1.4, U1.3 (VI)
- net V_Fuse: now also J7.3
- no-connect marks 33 -> 31
Other:
- moved on the sheet: C7, D1, D2, J5, J6, R1

Commit message: PCB Connected
Parts:
- removed C1, C3, C4: 10u, Capacitor_SMD:C_0805_2012Metric, symbol Device:C
- removed C11, C12, C13, C8: 100nF, Capacitor_SMD:C_0402_1005Metric, symbol Device:C
- removed C14: 4.7uF, Capacitor_SMD:C_0402_1005Metric, symbol Device:C
- removed C15: 2.2uF, Capacitor_SMD:C_0402_1005Metric, symbol Device:C
- removed C2: 22u, Capacitor_SMD:C_0805_2012Metric, symbol Device:C
- removed C5, C6: 1u, Capacitor_SMD:C_0402_1005Metric, symbol Device:C
- removed C7: 100n, Capacitor_SMD:C_0402_1005Metric, symbol Device:C
- removed C9: 1uF, Capacitor_SMD:C_0402_1005Metric, symbol Device:C
- removed D1, D2: MMBZ27VCLT1G, CMR_Voltage_Suppressor:SOT95P237X111-3N, symbol CMR_Voltage_Suppressor:MMBZ27VCLT1G
- removed D3, D4: GREEN, LED_SMD:LED_0603_1608Metric, symbol Device:LED
- removed F1: 3568, CMR_Fuse:FUSE_3568, symbol CMR_Fuse:3568
- removed J1: 3007W2PAT73A10X, CMR_Power_CAN_Connector:3007W2PAT73A10X, symbol CMR_Power_CAN_Connector:3007W2PAT73A10X
- removed J10, J11, J12, J13, J14, J9: 22232031, CMR_Fan_Pin_Header:CONN_A-6373-03A_MOL, symbol CMR_Fan_Pin_Header:22232031
- removed J2: Conn_01x02_Socket, Connector_AMASS:AMASS_XT30PW-M_1x02_P2.50mm_Horizontal, symbol Connector:Conn_01x02_Socket
- removed J3: Conn_01x03_Socket, Connector_JST:JST_PH_S3B-PH-SM4-TB_1x03-1MP_P2.00mm_Horizontal, symbol Connector:Conn_01x03_Socket
- removed J4: Conn_ARM_JTAG_SWD_10, Connector_PinHeader_1.27mm:PinHeader_2x05_P1.27mm_Vertical, symbol Connector:Conn_ARM_JTAG_SWD_10
- removed J5, J6: Conn_01x02_Pin, Connector_PinHeader_2.54mm:PinHeader_1x02_P2.54mm_Vertical, symbol Connector:Conn_01x02_Pin
- removed J7: 54-00236, CMR_LED_Array_Pins:TENSILITY_54-00236, symbol CMR_LED_Array_Pins:54-00236
- removed R1: 10k, Resistor_SMD:R_0402_1005Metric, symbol Device:R
- removed R10, R11, R12, R2, R3, R5, R6, R7, R8, R9: 1k, Resistor_SMD:R_0402_1005Metric, symbol Device:R
- removed TP1, TP2, TP3, TP4, TP5, TP6, TP7: TestPoint, TestPoint:TestPoint_Pad_D1.0mm, symbol Connector:TestPoint
- removed U1: AMS1117-5.0, Package_TO_SOT_SMD:SOT-223-3_TabPin2, symbol Regulator_Linear:AMS1117-5.0
- removed U2: AMS1117-3.3, Package_TO_SOT_SMD:SOT-223-3_TabPin2, symbol Regulator_Linear:AMS1117-3.3
- removed U3: TCAN1057AEV-Q1, Package_SO:SOIC-8_3.9x4.9mm_P1.27mm, symbol moteus:TCAN1042HGVDRBRQ1
- removed U4: STM32G431CBT6, Package_QFP:LQFP-48_7x7mm_P0.5mm, symbol MCU_ST_STM32G4:STM32G431CBTx
- removed U5, U6: CSD88537ND, CMR_N_Channel_Power_Mosfet:CSD88537ND8-M, symbol CMR_N_Channel_Power_Mosfet:CSD88537ND
Connections:
- no-connect marks 31 -> 0
Other:
- added sheet CAN (CAN.kicad_sch)
- added sheet Fan_Connectors (Fan_Connectors.kicad_sch)
- added sheet LED (LED.kicad_sch)
- added sheet MCU (MCU.kicad_sch)
- added sheet Power (Power.kicad_sch)
- added sheet Test_Points (Test_Points.kicad_sch)
