File: 2024-2025_Boards/LED_Board/Test_Points.kicad_sch (KiCad schematic)
At the start: 21 parts

Commit message: Board fixes
Parts:
- added D8, D9: YELLOW, LED_SMD:LED_0603_1608Metric, symbol Device:LED
- added R17: 2k, Resistor_SMD:R_0402_1005Metric, symbol Device:R
- added R18: 10k, Resistor_SMD:R_0402_1005Metric, symbol Device:R
- D3: value RED -> YELLOW
- TP1: value TestPoint -> GND
- TP2: value TestPoint -> LED1
- TP3: value TestPoint -> 5V
- TP4: value TestPoint -> LED2
- TP5: value TestPoint -> 3.3V
- TP6: value TestPoint -> LED3
- TP7: value TestPoint -> LED4
Connections:
- net 5V: now also D8.2 (A)
- net GND: now also R17.2, R18.2
- new net: D9.1 (K), R18.1
- new net: D8.1 (K), R17.1
- new net V_Fuse: D9.2 (A)
Other:
- moved on the sheet: D3, D4, D5, D6, D7, R12, R13, R14, R15, R16
