File: 2024-2025_Boards/LED_Board/CAN.kicad_sch (KiCad schematic)
At the start: 5 parts, among them U4 TCAN1057AEV-Q1

Commit message: Symbol library fix
Parts:
- D1, D2: footprint Cornell_Mars_Rover:SOT95P237X111-3N -> MMBZ27VCLT1G:SOT95P237X111-3N; symbol CMR_Voltage_Suppressor:MMBZ27VCLT1G -> Cornell_Mars_Rover:MMBZ27VCLT1G
Changed lines of the file:
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@@
 	)
 	(symbol
-		(lib_id "CMR_Voltage_Suppressor:MMBZ27VCLT1G")
+		(lib_id "Cornell_Mars_Rover:MMBZ27VCLT1G")
 		(at 165.1 113.03 0)
 		(unit 1)
@@
 			)
 		)
-		(property "Footprint" "Cornell_Mars_Rover:SOT95P237X111-3N"
+		(property "Footprint" "MMBZ27VCLT1G:SOT95P237X111-3N"
 			(at 165.1 113.03 0)
 			(effects
@@
 	)
 	(symbol
-		(lib_id "CMR_Voltage_Suppressor:MMBZ27VCLT1G")
+		(lib_id "Cornell_Mars_Rover:MMBZ27VCLT1G")
 		(at 118.11 113.03 0)
 		(unit 1)
@@
 			)
 		)
-		(property "Footprint" "Cornell_Mars_Rover:SOT95P237X111-3N"
+		(property "Footprint" "MMBZ27VCLT1G:SOT95P237X111-3N"
 			(at 118.11 113.03 0)
 			(effects
