File: 2024-2025_Boards/LED_Board/Power.kicad_sch (KiCad schematic)
At the start: 13 parts, among them J1 Conn_02x10_Odd_Even, U1 TLVM23625RDNR, U2 AMS1117-3.3

Commit message: Symbol library fix
Parts:
- F1: footprint Cornell_Mars_Rover:FUSE_3568 -> 3568:FUSE_3568; symbol CMR_Fuse:3568 -> Cornell_Mars_Rover:3568
- U1: footprint Cornell_Mars_Rover:RDN0011A-MFG -> TLVM23625RDNR:CONV_TLVM23625RDNR; symbol CMR_TLVM23625RDNR:TLVM23625RDNR -> Cornell_Mars_Rover:TLVM23625RDNR
Changed lines of the file:
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@@
 	)
 	(symbol
-		(lib_id "CMR_TLVM23625RDNR:TLVM23625RDNR")
+		(lib_id "Cornell_Mars_Rover:TLVM23625RDNR")
 		(at 142.24 118.11 0)
 		(unit 1)
@@
 			)
 		)
-		(property "Footprint" "Cornell_Mars_Rover:RDN0011A-MFG"
+		(property "Footprint" "TLVM23625RDNR:CONV_TLVM23625RDNR"
 			(at 142.24 118.11 0)
 			(effects
@@
 	)
 	(symbol
-		(lib_id "CMR_Fuse:3568")
+		(lib_id "Cornell_Mars_Rover:3568")
 		(at 146.05 59.69 0)
 		(unit 1)
@@
 			)
 		)
-		(property "Footprint" "Cornell_Mars_Rover:FUSE_3568"
+		(property "Footprint" "3568:FUSE_3568"
 			(at 145.542 52.832 0)
 			(effects
