File: 2025-2026_Boards/otto_onboarding_stuff/KiCad_Tutorial.kicad_pcb (KiCad board)
At the start: 2 copper layers, 28 parts, among them J1 USB_B_Micro, J2 Conn_01x04_Pin, J3 Conn_01x04_Pin, J4 Conn_01x04_Pin, SW1 SW_SPDT, U1 STM32F103C8T6, U3 AMS1117-3.3, Y1 16MHz

Commit message: Worked on wiring.
Parts:
- added H1: MountingHole, MountingHole:MountingHole_2.2mm_M2, F.Cu at (89.5, 64.0)
- added H2: MountingHole, MountingHole:MountingHole_2.2mm_M2, F.Cu at (128.0, 62.0)
- added H3: MountingHole, MountingHole:MountingHole_2.2mm_M2, F.Cu at (89.5, 88.0)
- added H4: MountingHole, MountingHole:MountingHole_2.2mm_M2, F.Cu at (109.0, 94.5)
- SW1: footprint Button_Switch_THT:SW_Lever_1P2T_NKK_GW12LxH -> Button_Switch_SMD:SW_SPDT_PCM12
- moved C7 13.6 mm to (107.5, 81.5), turned to 0 degrees
- moved D1 12.7 mm to (105.2, 80.5), turned to 180 degrees
- moved C5 12.5 mm to (107.5, 73.5)
- moved SW1 12.2 mm to (96.3, 66.5), turned to -90 degrees
- moved R1 10.5 mm to (107.0, 80.5)
- moved J2 10.2 mm to (106.5, 70.3), turned to 180 degrees
- moved R3 9.85 mm to (107.5, 79.0), turned to 180 degrees
- moved C2 9.15 mm to (105.5, 83.0), turned to -90 degrees
- moved J4 7.11 mm to (97.4, 87.0), turned to 90 degrees
- moved U3 6.79 mm to (113.8, 84.5)
- moved J3 5.50 mm to (110.5, 70.9)
- moved C1 5.41 mm to (108.2, 85.0), turned to 90 degrees
- moved C9 4.92 mm to (97.0, 83.0)
- moved J1 4.71 mm to (118.5, 73.7)
- moved Y1 3.91 mm to (92.4, 75.8), turned to 180 degrees
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Routing:
- net +3.3V: track 0.00 -> 54.5 mm
- net VBUS: track 0.00 -> 26.7 mm
- net GND: track 0.00 -> 22.8 mm, vias 0 -> 6
- net /USB_D+: track 0.00 -> 19.9 mm
- net /USART1_RX: track 0.00 -> 12.3 mm
- net /SDIO: track 0.00 -> 12.2 mm
- net /HSE_OUT: track 0.00 -> 10.2 mm
- net /USART1_TX: track 0.00 -> 9.27 mm
- net /SWCLK: track 0.00 -> 8.92 mm
- net /I2C2_STA: track 0.00 -> 8.34 mm
- net /I2C2_STL: track 0.00 -> 5.86 mm
- net /NRST: track 0.00 -> 5.81 mm
- net +3.3VA: track 0.00 -> 5.70 mm
- net /BOOT0: track 0.00 -> 4.08 mm
- net /HSE_IN: track 0.00 -> 3.83 mm
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- added copper zone on B.Cu, net GND
Other:
- board outline added: 38.5 x 29.5 mm

Commit message: almost finished wiring. gonna hook up grounds later
Parts:
- moved J2 2.82 mm to (104.0, 69.0)
- moved J1 1.85 mm to (117.9, 75.5), turned to 180 degrees
- moved J3 1.70 mm to (111.0, 72.5), turned to 180 degrees
- moved C13 0.50 mm to (95.0, 77.0), turned to 90 degrees
- moved Y1 0.50 mm to (91.9, 75.8)
Routing:
- net +3.3V: track 54.5 -> 81.3 mm
- net /USB_D-: track 0.00 -> 14.5 mm
- net GND: track 22.8 -> 31.9 mm, vias 6 -> 5
- net VBUS: track 26.7 -> 20.2 mm
- net +3.3VA: track 5.70 -> 10.1 mm
- net /SDIO: track 12.2 -> 8.40 mm
- net /USART1_RX: track 12.3 -> 9.50 mm
- net /USART1_TX: track 9.27 -> 6.75 mm
- net /HSE_OUT: track 10.2 -> 7.79 mm
- net /USB_D+: track 19.9 -> 21.2 mm
- net /HSE_IN: track 3.83 -> 4.33 mm

Commit message: completed(-ish) onboarding project
Parts:
- moved H4 13.6 mm to (121.0, 88.0)
- moved H2 7.07 mm to (121.0, 63.0)
- moved SW1 0.65 mm to (96.3, 65.8)
Routing:
- net GND: track 31.9 -> 45.1 mm, vias 5 -> 10
- net /USB_D+: track 21.2 -> 23.8 mm
- net +3.3V: track 81.3 -> 81.9 mm
Other:
- board size 38.5 x 29.5 mm -> 36.5 x 31.7 mm
Changed lines of the file:
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@@
 	(footprint "MountingHole:MountingHole_2.2mm_M2"
 		(layer "F.Cu")
-		(at 128 62)
+		(at 121 63)
 		(descr "Mounting Hole 2.2mm, M2, no annular, generated by kicad-footprint-generator mountinghole.py")
 		(tags "mountinghole M2")
@@
 		(tags "Through hole pin header THT 1x04 2.54mm single row")
 		(property "Reference" "J2"
-			(at 0 10.04 0)
+			(at -2.5 8.5 0)
 			(layer "F.SilkS")
 			(effects
@@
 	(footprint "MountingHole:MountingHole_2.2mm_M2"
 		(layer "F.Cu")
-		(at 109 94.5)
+		(at 121 88)
 		(descr "Mounting Hole 2.2mm, M2, no annular, generated by kicad-footprint-generator mountinghole.py")
 		(tags "mountinghole M2")
@@
 	(footprint "Button_Switch_SMD:SW_SPDT_PCM12"
 		(layer "F.Cu")
-		(at 96.33 66.5 -90)
+		(at 96.33 65.85 -90)
 		(descr "Ultraminiature Surface Mount Slide Switch, right-angle, https://www.ckswitches.com/media/1424/pcm.pdf")
 		(property "Reference" "SW1"
@@
 	)
 	(gr_arc
-		(start 121.5 61.5)
-		(mid 122.914214 62.085786)
-		(end 123.5 63.5)
+		(start 121.414214 58.914215)
+		(mid 122.884851 59.468689)
+		(end 123.501838 60.914214)
 		(stroke
 			(width 0.2)
@@
 	)
 	(gr_line
-		(start 97.951496 60.0355)
-		(end 130.451496 60.0355)
+		(start 88.914214 58.914215)
+		(end 121.414214 58.914215)
 		(stroke
 			(width 0.2)
@@
 		)
 		(layer "F.Cu")
-		(net 19)
+		(net 4)
 	)
 	(gr_arc
@@
 	(gr_line
 		(start 87 88)
-		(end 87 63.5)
+		(end 86.914215 60.914214)
 		(stroke
 			(width 0.2)
@@
 	)
 	(gr_arc
-		(start 87 63.5)
-		(mid 87.585786 62.085786)
-		(end 89 61.5)
+		(start 86.914214 60.914214)
+		(mid 87.5 59.5)
+		(end 88.914214 58.914214)
 		(stroke
 			(width 0.2)
@@
 	)
 	(gr_line
-		(start 123.5 63.5)
+		(start 123.5 60.914214)
 		(end 123.5 88.5)
 		(stroke
@@
 	)
 	(gr_arc
-		(start 121.5 61.5)
-		(mid 122.914214 62.085786)
-		(end 123.5 63.5)
+		(start 121.507595 58.83052)
+		(mid 122.921742 59.472734)
+		(end 123.5 60.914215)
 		(stroke
 			(width 0.05)
@@
 	(gr_line
 		(start 87 88)
-		(end 87 63.5)
+		(end 87 60.9142)
 		(stroke
 			(width 0.05)
@@
 	)
 	(gr_arc
-		(start 87 63.5)
-		(mid 87.585786 62.085786)
-		(end 89 61.5)
+		(start 87 60.914214)
+		(mid 87.585786 59.5)
+		(end 89 58.914214)
 		(stroke
 			(width 0.05)
@@
 	(gr_line
 		(start 123.5 64)
-		(end 123.5 63.5)
+		(end 123.5 60.914215)
 		(stroke
 			(width 0.05)
@@
 	)
 	(gr_line
-		(start 93 61)
-		(end 125.5 61)
+		(start 88.25 59)
+		(end 120.75 59)
 		(stroke
 			(width 0.05)
@@
 	)
 	(segment
-		(start 110.5 88.5)
-		(end 110.7 88.3)
-		(width 0.3)
-		(layer "F.Cu")
-		(net 1)
-	)
-	(segment
 		(start 117.810768 86.8)
 		(end 119.175 85.435768)
@@
 	)
 	(segment
+		(start 96.54 72)
+		(end 96.54 71.165997)
+		(width 0.3)
+		(layer "F.Cu")
+		(net 2)
+	)
+	(segment
 		(start 105.5 73)
 		(end 105.9375 73)
@@
 	)
 	(segment
+		(start 116.575 77.35)
+		(end 116.575 78.275)
+		(width 0.2)
+		(layer "F.Cu")
+		(net 2)
+	)
+	(segment
 		(start 94.835 72.5)
 		(end 94.835 71.795)
@@
 	)
 	(segment
+		(start 99 64)
+		(end 99.5 64)
+		(width 0.3)
+		(layer "F.Cu")
+		(net 2)
+	)
+	(segment
 		(start 104 73.5)
 		(end 104.017034 73.5)
@@
 	)
 	(segment
+		(start 99 71)
+		(end 99.5 70.5)
+		(width 0.2)
+		(layer "F.Cu")
+		(net 2)
+	)
+	(segment
+		(start 104 61.38)
+		(end 102.12 61.38)
+		(width 0.2)
+		(layer "F.Cu")
+		(net 2)
+	)
+	(segment
 		(start 93 76.7)
 		(end 94.82 76.7)
@@
 	)
 	(segment
+		(start 96.54 71.165997)
+		(end 96.452751 71.078748)
+		(width 0.3)
+		(layer "F.Cu")
+		(net 2)
+	)
+	(segment
+		(start 99 72.175)
+		(end 99 71)
+		(width 0.2)
+		(layer "F.Cu")
+		(net 2)
+	)
+	(segment
 		(start 104.517034 73)
 		(end 105.5 73)
@@
 	)
 	(segment
+		(start 116.575 78.275)
+		(end 115 79.85)
+		(width 0.2)
+		(layer "F.Cu")
+		(net 2)
+	)
+	(segment
+		(start 97.76 64.25)
+		(end 97.76 63.6)
+		(width 0.3)
+		(layer "F.Cu")
+		(net 2)
+	)
+	(segment
+		(start 102.12 61.38)
+		(end 101.5 62)
+		(width 0.2)
+		(layer "F.Cu")
+		(net 2)
+	)
+	(segment
 		(start 107.96 72.54)
 		(end 108 72.5)
@@
 	)
 	(segment
+		(start 111 64.88)
+		(end 110.12 64)
+		(width 0.2)
+		(layer "F.Cu")
+		(net 2)
+	)
+	(segment
+		(start 110.12 64)
+		(end 108.5 64)
+		(width 0.2)
+		(layer "F.Cu")
+		(net 2)
+	)
+	(segment
 		(start 94.835 71.795)
 		(end 94.54 71.5)
@@
 	)
 	(via
+		(at 96.452751 71.078748)
+		(size 0.6)
+		(drill 0.3)
+		(layers "F.Cu" "B.Cu")
+		(net 2)
+	)
+	(via
 		(at 106 72.9375)
 		(size 0.6)
@@
 	)
 	(via
+		(at 115 79.85)
+		(size 0.6)
+		(drill 0.3)
+		(layers "F.Cu" "B.Cu")
+		(net 2)
+	)
+	(via
+		(at 99.5 70.5)
+		(size 0.6)
+		(drill 0.3)
+		(layers "F.Cu" "B.Cu")
+		(net 2)
+	)
+	(via
+		(at 101.5 62)
+		(size 0.6)
+		(drill 0.3)
+		(layers "F.Cu" "B.Cu")
+		(net 2)
+	)
+	(via
 		(at 90 73.5)
 		(size 0.6)
@@
 	)
 	(via
-		(at 99 64)
+		(at 108.5 64)
+		(size 0.6)
+		(drill 0.3)
+		(layers "F.Cu" "B.Cu")
+		(net 2)
+	)
+	(via
+		(at 99.5 64)
 		(size 0.6)
 		(drill 0.3)
@@
 	)
 	(segment
+		(start 115 79.85)
+		(end 115.35 79.5)
+		(width 0.2)
+		(layer "B.Cu")
+		(net 2)
+	)
+	(segment
 		(start 104.835 80.5)
 		(end 104 80.5)
@@
 	)
 	(segment
-		(start 98.5 69.49)
-		(end 97.76 68.75)
-		(width 0.3)
-		(layer "F.Cu")
-		(net 3)
-	)
-	(segment
 		(start 111.497471 68.759)
 		(end 110.502529 68.759)
@@
 	)
 	(segment
+		(start 98.5 69.49)
+		(end 97.76 68.75)
+		(width 0.3)
+		(layer "F.Cu")
+		(net 3)
+	)
+	(segment
 		(start 104.835 81.435)
 		(end 105.5 82.1)
@@
 	)
 	(segment
+		(start 97.76 68.75)
+		(end 97.76 68.1)
+		(width 0.3)
+		(layer "F.Cu")
+		(net 3)
+	)
+	(segment
 		(start 95.475 72.5)
 		(end 95.475 71.525)
@@
 	)
 	(segment
-		(start 104.571466 79.5885)
-		(end 106.3915 79.5885)
+		(start 110.51105 80.5)
+		(end 117.5 80.5)
 		(width 0.3)
 		(layer "F.Cu")
@@
 	)
 	(segment
-		(start 108.66205 78.651)
-		(end 117.599 78.651)
+		(start 104.571466 79.5885)
+		(end 106.3915 79.5885)
 		(width 0.3)
 		(layer "F.Cu")
@@
 	)
 	(segment
-		(start 117.875 78.375)
-		(end 117.875 77.35)
+		(start 117.5 80.5)
+		(end 117.5 78.75)
 		(width 0.3)
 		(layer "F.Cu")
@@
 	)
 	(segment
+		(start 108.34005 78.329)
+		(end 110.51105 80.5)
+		(width 0.3)
+		(layer "F.Cu")
+		(net 12)
+	)
+	(segment
 		(start 105.4125 75.0875)
 		(end 104.4125 75.0875)
@@
 	)
 	(segment
-		(start 106.98 79)
-		(end 107.651 78.329)
+		(start 117.5 78.75)
+		(end 117.875 78.375)
 		(width 0.3)
 		(layer "F.Cu")
@@
 	)
 	(segment
-		(start 107.651 78.329)
-		(end 108.34005 78.329)
+		(start 106.3915 79.5885)
+		(end 106.98 79)
 		(width 0.3)
 		(layer "F.Cu")
@@
 	)
 	(segment
-		(start 117.599 78.651)
-		(end 117.875 78.375)
+		(start 106.98 79)
+		(end 107.651 78.329)
 		(width 0.3)
 		(layer "F.Cu")
@@
 	)
 	(segment
-		(start 106.3915 79.5885)
-		(end 106.98 79)
+		(start 104 75.5)
+		(end 104 79.4115)
 		(width 0.3)
 		(layer "F.Cu")
@@
 	)
 	(segment
-		(start 108.34005 78.329)
-		(end 108.66205 78.651)
+		(start 107.651 78.329)
+		(end 108.34005 78.329)
 		(width 0.3)
 		(layer "F.Cu")
@@
 	)
 	(segment
-		(start 104 75.5)
-		(end 104 79.4115)
+		(start 117.875 78.375)
+		(end 117.875 77.35)
 		(width 0.3)
 		(layer "F.Cu")
@@
 	)
 	(segment
-		(start 97.76 67.25)
-		(end 99.26 67.25)
-		(width 0.5)
+		(start 98.61 66.6)
+		(end 97.76 66.6)
+		(width 0.2)
 		(layer "F.Cu")
 		(net 24)
 	)
 	(segment
-		(start 99.26 67.25)
-		(end 99.5 67.49)
-		(width 0.5)
+		(start 99.5 67.49)
+		(end 98.61 66.6)
+		(width 0.2)
 		(layer "F.Cu")
 		(net 24)
@@
 		(polygon
 			(pts
-				(xy 87 62.069661) (xy 123.5 62.069661) (xy 123.5 91.069661) (xy 86.5 90.5)
+				(xy 87 59) (xy 123.5 59) (xy 123.5 91.069661) (xy 86.5 90.5)
 			)
 		)
