File: 2025-2026_Boards/Mars Rover Onboarding/Mars Rover Onboarding.kicad_pcb (KiCad board)
At the start: 2 copper layers, 0 parts

Commit message: Onboarding
Parts:
- added C1: 22u, Capacitor_SMD:C_0805_2012Metric, F.Cu at (94.0, 82.0)
- added C10: 1u, Capacitor_SMD:C_0402_1005Metric, F.Cu at (78.0, 84.0)
- added C11: 100n, Capacitor_SMD:C_0402_1005Metric, F.Cu at (83.0, 83.5)
- added C12: 10p, Capacitor_SMD:C_0402_1005Metric, F.Cu at (76.5, 76.2)
- added C13: 10p, Capacitor_SMD:C_0402_1005Metric, F.Cu at (76.5, 78.2)
- added C2: 22u, Capacitor_SMD:C_0805_2012Metric, F.Cu at (100.0, 88.5)
- added C3: 10u, Capacitor_SMD:C_0603_1608Metric, F.Cu at (82.5, 69.8)
- added C4: 100n, Capacitor_SMD:C_0402_1005Metric, F.Cu at (79.0, 74.2)
- added C5: 100n, Capacitor_SMD:C_0402_1005Metric, F.Cu at (88.0, 83.8)
- added C6: 100n, Capacitor_SMD:C_0402_1005Metric, F.Cu at (91.0, 75.0)
- added C7: 100n, Capacitor_SMD:C_0402_1005Metric, F.Cu at (82.5, 71.5)
- added C8: 10n, Capacitor_SMD:C_0402_1005Metric, F.Cu at (79.0, 78.5)
- added C9: 1u, Capacitor_SMD:C_0402_1005Metric, F.Cu at (78.0, 82.5)
- added D1: RED, LED_SMD:LED_0603_1608Metric, F.Cu at (103.0, 88.5)
- added FB1: 120R, Inductor_SMD:L_0603_1608Metric, F.Cu at (80.0, 83.0)
- added H1: MountingHole, MountingHole:MountingHole_2.2mm_M2, F.Cu at (68.2, 94.8)
- added H2: MountingHole, MountingHole:MountingHole_2.2mm_M2, F.Cu at (104.2, 94.8)
- added H3: MountingHole, MountingHole:MountingHole_2.2mm_M2, F.Cu at (104.2, 64.2)
- added H4: MountingHole, MountingHole:MountingHole_2.2mm_M2, F.Cu at (68.2, 64.2)
- added J1: USB_B_Micro, Connector_USB:USB_Micro-B_Wuerth_629105150521, F.Cu at (103.0, 77.0)
- added J2: Conn_01x04_Pin, Connector_PinHeader_2.54mm:PinHeader_1x04_P2.54mm_Vertical, F.Cu at (83.6, 63.5)
- added J3: Conn_01x04_Pin, Connector_PinHeader_2.54mm:PinHeader_1x04_P2.54mm_Vertical, F.Cu at (97.6, 63.5)
- added J4: Conn_01x04_Pin, Connector_PinHeader_2.54mm:PinHeader_1x04_P2.54mm_Vertical, F.Cu at (78.4, 95.2)
- added R1: 1k5, Resistor_SMD:R_0402_1005Metric, F.Cu at (103.5, 85.8)
- added R2: 10k, Resistor_SMD:R_0402_1005Metric, F.Cu at (71.5, 72.5)
- added R3: 1k5, Resistor_SMD:R_0402_1005Metric, F.Cu at (94.8, 75.0)
- added R4: 1k5, Resistor_SMD:R_0402_1005Metric, F.Cu at (82.0, 90.8)
- added R5: 1k5, Resistor_SMD:R_0402_1005Metric, F.Cu at (84.5, 90.8)
- added SW1: SW_SPDT, Button_Switch_SMD:SW_SPDT_PCM12, F.Cu at (67.8, 72.8)
- added U1: AMS1117-3.3, Package_TO_SOT_SMD:SOT-223-3_TabPin2, F.Cu at (95.0, 88.0)
- added U2: STM32F103C8T6, Package_QFP:LQFP-48_7x7mm_P0.5mm, F.Cu at (85.0, 77.5)
- added Y1: 16MHz, Crystal:Crystal_SMD_3225-4Pin_3.2x2.5mm, F.Cu at (74.0, 77.0)
Routing:
- net +3.3V: track 0.00 -> 183.3 mm, vias 0 -> 6
- net GND: track 0.00 -> 28.6 mm, vias 0 -> 20
- net /SW_BOOT0: track 0.00 -> 23.8 mm
- net /SWDIO: track 0.00 -> 16.4 mm
- net /I2C2_SCL: track 0.00 -> 15.8 mm
- net /I2C2_SDA: track 0.00 -> 14.9 mm
- net /USART1_RX: track 0.00 -> 14.1 mm
- net /USB_D+: track 0.00 -> 12.9 mm
- net /USB_D-: track 0.00 -> 12.3 mm
- net /USART1_TX: track 0.00 -> 12.0 mm
- net /SWCLK: track 0.00 -> 11.8 mm
- net /NRST: track 0.00 -> 9.93 mm
- net /HSE_IN: track 0.00 -> 8.64 mm
- net +3.3VA: track 0.00 -> 7.31 mm
- net /HSE_OUT: track 0.00 -> 7.22 mm
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- added copper zone on F.Cu, net +3.3V
- added copper zone on B.Cu, net GND
- added copper zone on F.Cu, net GND
- added copper zone on F.Cu, net VBUS
Other:
- board outline added: 42 x 36.5 mm
- board text added: "BOOT"
- board text added: "I2C"
- board text added: "ON"
- board text added: "SWD"
- board text added: "UART"
- board text added: "USB"
