File: 2025-2026_Boards/Mars Rover Onboarding/Mars Rover Onboarding.kicad_sch (KiCad schematic)
At the start: 28 parts, among them J1 USB_B_Micro, J2 Conn_01x04_Pin, J3 Conn_01x04_Pin, J4 Conn_01x04_Pin, SW1 SW_SPDT, U1 STM32F103C8T6, U2 AMS1117-3.3, Y1 16MHz

Commit message: Onboarding
Parts:
- added H1, H2, H3, H4: MountingHole, MountingHole:MountingHole_2.2mm_M2, symbol Mechanical:MountingHole
- SW1: footprint Button_Switch_THT:SW_E-Switch_EG1224_SPDT_Angled -> Button_Switch_SMD:SW_SPDT_PCM12
- renumbered C12 to C1, C8 to C10, C9 to C11, C10 to C12, C11 to C13, C13 to C2, C5 to C3, C3 to C5, C2 to C6, C1 to C7, C6 to C8, C7 to C9, J3 to J2, J2 to J3, R3 to R1, R1 to R2, R2 to R3, U2 to U1, U1 to U2
Other:
- note added: "M2"
- note added: "Mounting Holes"
