File: 2025-2026_Boards/temperature_board/TEMPERATURE_SENSOR_KICAD/_autosave-TEMPERATURE_SENSOR_KICAD.kicad_sch (KiCad schematic)
At the start: 39 parts, among them U1 STM32G431CBT6, U2 TMP235A4DBZR, U3 AMS1117-3.3, U4 TPS54240DGQ

Commit message: minor edits
Parts:
- L1: value L -> 10u
Changed lines of the file:
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@@
 		)
 	)
+	(text "FAN SYSTEMS \nAND POWER SUPPLY\n"
+		(exclude_from_sim no)
+		(at 82.296 172.974 0)
+		(effects
+			(font
+				(size 2.54 2.54)
+			)
+			(justify left)
+		)
+	)
 	(text "1 x 100nF Capacitor per Pin"
 		(exclude_from_sim no)
@@
 			)
 		)
-		(property "Value" "L"
+		(property "Value" "10u"
 			(at 116.84 21.59 90)
 			(effects
