File: 2025-2026_Boards/temperature_board/TEMPERATURE_SENSOR_KICAD/_autosave-TEMPERATURE_SENSOR_KICAD.kicad_sch (KiCad schematic)
At the start: 79 parts, among them J1 LCD Connector Pinout, Q1 Q_NPN_BCE, Q3 Q_NPN_BCE, Q4 Q_NPN_BCE, Q5 Q_PNP_BCE, U1 STM32G431CBT6, U2 TMP235A4DBZR, U3 AMS1117-3.3, U5 TPS62932DRLR, U8 AMS1117

Commit message: finished pcb hopefully forever
Parts:
- U5: footprint SOT8_DRL_TEX -> (none)
Changed lines of the file:
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@@
 			)
 		)
-		(property "Footprint" "SOT8_DRL_TEX"
+		(property "Footprint" ""
 			(at 181.61 40.64 0)
 			(effects
