File: 2025-2026_Boards/temperature_board/TEMPERATURE_SENSOR_KICAD/_autosave-TEMPERATURE_SENSOR_KICAD.kicad_pcb (KiCad board)
At the start: 2 copper layers, 73.3 x 75.8 mm, 89 parts, among them J1 LCD Connector Pinout, J10 Conn_01x02_Pin, J11 Conn_01x02_Pin, J12 Conn_01x02_Pin, J13 Conn_01x02_Pin, J14 Conn_01x02_Pin, J15 Conn_01x02_Pin, J16 Conn_01x02_Pin, J17 Conn_01x02_Pin, J18 Conn_01x02_Pin, J19 Conn_01x02_Pin, J2 Conn_01x02_Pin, J20 Conn_01x02_Pin, J21 Conn_01x02_Pin, J22 Conn_01x02_Pin, J23 Conn_01x02_Pin, J24 Conn_01x03_Socket, J25 Conn_01x03_Socket, J3 Conn_01x02_Pin, J4 Conn_01x02_Pin, J5 Conn_01x02_Pin, J6 Conn_01x02_Pin, J7 Conn_01x02_Pin, J8 Conn_01x02_Pin, J9 Conn_01x02_Pin, Q1 Q_NPN_BCE, Q3 Q_NPN_BCE, Q4 Q_NPN_BCE, Q5 Q_PNP_BCE, U1 STM32G431CBT6, U2 TMP235A4DBZR, U3 AMS1117-3.3, U4 TCAN1057AEV-Q1, U5 TPS62932DRLR

Commit message: rehashed
Parts:
- removed the TP1 at (97.5, 132.0)
- moved R1 39.1 mm to (127.8, 142.0), turned to 90 degrees
- moved D1 38.3 mm to (126.6, 142.5), turned to 180 degrees
- moved C2 38.2 mm to (127.6, 144.6), turned to 0 degrees
- moved TP1 38.2 mm to (128.2, 138.3)
- moved C1 29.5 mm to (117.6, 147.6)
- moved Rfbb1 29.4 mm to (98.2, 118.3)
- moved Cin4 28.6 mm to (92.5, 120.3), turned to -90 degrees
- moved L2 28.3 mm to (94.7, 130.0)
- moved Q4 28.0 mm to (127.7, 130.1), turned to -90 degrees
- moved Css2 27.4 mm to (98.7, 119.8), turned to 90 degrees
- moved U3 27.4 mm to (121.3, 142.0)
- moved Rfbt1 26.8 mm to (100.8, 121.2)
- moved U5 26.2 mm to (96.4, 120.7), turned to 0 degrees
- moved Q5 25.7 mm to (130.6, 130.1), turned to -90 degrees
- moved R10 25.2 mm to (128.4, 133.2), turned to 90 degrees
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Routing:
- net Net-(J1-Pin_12): track 83.0 -> 12.0 mm
- net Net-(U1-PA10): track 55.3 -> 3.04 mm
- net Net-(J1-Pin_8): track 61.1 -> 23.0 mm, vias 0 -> 4
- net Net-(J1-Pin_9): track 50.7 -> 13.9 mm
- net Net-(U1-PA8): track 40.5 -> 10.2 mm, vias 2 -> 0
- net 28V: track 58.7 -> 31.4 mm, vias 1 -> 0
- net Net-(J1-Pin_10): track 9.64 -> 34.6 mm, vias 0 -> 2
- net Net-(U1-PA7): track 21.9 -> 1.55 mm, vias 2 -> 0
- net Net-(J1-Pin_6): track 43.2 -> 26.1 mm
- net Net-(U1-PA14): track 12.9 -> 24.2 mm, vias 0 -> 4
- net Net-(U1-PA6): track 14.5 -> 23.1 mm, vias 0 -> 2
- net Net-(J1-Pin_11): track 17.5 -> 26.0 mm, vias 0 -> 4
- net Net-(Q3-B): track 1.65 -> 9.75 mm, vias 0 -> 4
- net Net-(U1-PA3): track 9.81 -> 3.07 mm
- net +3.3V: track 112.8 -> 119.0 mm, vias 10 -> 14
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Other:
- board text removed: "100n"
