File: 2025-2026_Boards/temperature_board/TEMPERATURE_SENSOR_KICAD/FAN_PINS.kicad_sch (KiCad schematic)
At the start: 27 parts, among them J10 Conn_01x02_Pin, J11 Conn_01x02_Pin, J12 Conn_01x02_Pin, J13 Conn_01x02_Pin, J14 Conn_01x02_Pin, J15 Conn_01x02_Pin, J16 Conn_01x02_Pin, J17 Conn_01x02_Pin, J18 Conn_01x02_Pin, J19 Conn_01x02_Pin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

Commit message: fixed can
Connections:
- net CAN+: now also J25.1 (Pin_1); no longer J25.2 (Pin_2)
- net CAN-: now also J25.2 (Pin_2); no longer J25.1 (Pin_1)
Changed lines of the file:
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@@
 	(paper "A4")
 	(junction
-		(at 245.11 71.12)
-		(diameter 0)
-		(color 0 0 0 0)
-	)
-	(junction
 		(at 234.95 73.66)
 		(diameter 0)
@@
 	)
 	(junction
+		(at 242.57 71.12)
+		(diameter 0)
+		(color 0 0 0 0)
+	)
+	(junction
 		(at 146.05 76.2)
 		(diameter 0)
@@
 	)
 	(junction
-		(at 242.57 73.66)
+		(at 245.11 73.66)
 		(diameter 0)
 		(color 0 0 0 0)
@@
 	(wire
 		(pts
-			(xy 234.95 73.66) (xy 242.57 73.66)
-		)
-		(stroke
-			(width 0)
-			(type default)
-		)
-	)
-	(wire
-		(pts
 			(xy 134.62 86.36) (xy 146.05 86.36)
 		)
@@
 	(wire
 		(pts
-			(xy 232.41 71.12) (xy 245.11 71.12)
-		)
-		(stroke
-			(width 0)
-			(type default)
-		)
-	)
-	(wire
-		(pts
 			(xy 231.14 91.44) (xy 231.14 76.2)
 		)
@@
 	(wire
 		(pts
-			(xy 245.11 71.12) (xy 245.11 83.82)
+			(xy 245.11 73.66) (xy 245.11 83.82)
 		)
 		(stroke
@@
 	(wire
 		(pts
-			(xy 242.57 73.66) (xy 251.46 73.66)
+			(xy 234.95 73.66) (xy 245.11 73.66)
 		)
 		(stroke
@@
 	(wire
 		(pts
-			(xy 242.57 73.66) (xy 242.57 81.28)
-		)
-		(stroke
-			(width 0)
-			(type default)
-		)
-	)
-	(wire
-		(pts
 			(xy 237.49 67.31) (xy 234.95 67.31)
 		)
@@
 	(wire
 		(pts
+			(xy 245.11 73.66) (xy 251.46 73.66)
+		)
+		(stroke
+			(width 0)
+			(type default)
+		)
+	)
+	(wire
+		(pts
+			(xy 242.57 71.12) (xy 242.57 81.28)
+		)
+		(stroke
+			(width 0)
+			(type default)
+		)
+	)
+	(wire
+		(pts
 			(xy 146.05 76.2) (xy 146.05 77.47)
 		)
@@
 	(wire
 		(pts
+			(xy 242.57 71.12) (xy 251.46 71.12)
+		)
+		(stroke
+			(width 0)
+			(type default)
+		)
+	)
+	(wire
+		(pts
 			(xy 251.46 81.28) (xy 242.57 81.28)
 		)
@@
 	(wire
 		(pts
-			(xy 245.11 71.12) (xy 251.46 71.12)
-		)
-		(stroke
+			(xy 232.41 71.12) (xy 242.57 71.12)
+		)
+		(stroke
