File: 2025-2026_Boards/FDCAN-USB_Board/CAN-FD.kicad_sch (KiCad schematic)
At the start: 10 parts, among them J2 Conn_01x03_Socket, J3 Conn_01x03_Socket, U4 TCAN1057AEV-Q1, U5 TCAN1057AEV-Q1

Commit message: Layout finished
Parts:
- added C13, C14: 1u, Capacitor_SMD:C_0402_1005Metric, symbol Device:C
- added J4: Conn_01x03_Socket, Connector_JST:JST_PH_S3B-PH-SM4-TB_1x03-1MP_P2.00mm_Horizontal, symbol Connector:Conn_01x03_Socket
- added R13: 120, Resistor_SMD:R_1206_3216Metric, symbol Device:R_US
- added U6: TCAN1057AEV-Q1, Package_SO:SOIC-8_3.9x4.9mm_P1.27mm, symbol Cornell_Mars_Rover:TCAN1057AEV-Q1
Connections:
- net 3.3V: now also C14.1, U6.5 (VIO)
- net 5V: now also C13.1, U6.3 (VCC)
- net GND: now also C13.2, C14.2, J4.3 (Pin_3), U6.2 (GND), U6.8 (STB)
- net CANH1 renamed CAN1+
- net CANH2 renamed CAN2+
- net CANL1 renamed CAN1-
- net CANL2 renamed CAN2-
- new net CAN3+: J4.1 (Pin_1), R13.1, U6.7 (CANH)
- new net CAN3-: J4.2 (Pin_2), R13.2, U6.6 (CANL)
- new net CAN_RX3: U6.4 (RXD)
- new net CAN_TX3: U6.1 (TXD)
