File: 2025-2026_Boards/FDCAN-USB_Board/LED_Debug.kicad_sch (KiCad schematic)
At the start: 23 parts

Commit message: Layout finished
Parts:
- added D5: GREEN, LED_SMD:LED_0603_1608Metric, symbol Device:LED
- added D8: YELLOW, LED_SMD:LED_0603_1608Metric, symbol Device:LED
- added R14, R15: 1k, Resistor_SMD:R_0402_1005Metric, symbol Device:R_US
- D10: renamed from D8; value YELLOW -> BLUE
- D6: renamed from D4; value GREEN -> YELLOW
- D7: renamed from D6; value GREEN -> YELLOW
- D9: renamed from D7; value YELLOW -> BLUE
- renumbered D5 to D4
Connections:
- net GND: now also R14.2, R15.2
- new net: D8.1 (K), R15.1
- new net: D5.1 (K), R14.1
- new net LED_RX_3: D8.2 (A)
- new net LED_TX_3: D5.2 (A)
Other:
- moved on the sheet: D1, D10, D2, D3, D4, D6, D7, D9, H1, H2, H3, H4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

Commit message: Gerber files, BOM, layout fix
Parts:
- R10, R11, R12, R14, R15, R5, R6, R7, R8, R9: value 1k -> 220
Changed lines of the file:
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@@
 			)
 		)
-		(property "Value" "1k"
+		(property "Value" "220"
 			(at 100.33 72.39 90)
 			(effects
@@
 			)
 		)
-		(property "Value" "1k"
+		(property "Value" "220"
 			(at 163.83 135.89 90)
 			(effects
@@
 			)
 		)
-		(property "Value" "1k"
+		(property "Value" "220"
 			(at 163.83 59.69 90)
 			(effects
@@
 			)
 		)
-		(property "Value" "1k"
+		(property "Value" "220"
 			(at 100.33 110.49 90)
 			(effects
@@
 			)
 		)
-		(property "Value" "1k"
+		(property "Value" "220"
 			(at 163.83 72.39 90)
 			(effects
@@
 			)
 		)
-		(property "Value" "1k"
+		(property "Value" "220"
 			(at 163.83 123.19 90)
 			(effects
@@
 			)
 		)
-		(property "Value" "1k"
+		(property "Value" "220"
 			(at 163.83 110.49 90)
 			(effects
@@
 			)
 		)
-		(property "Value" "1k"
+		(property "Value" "220"
 			(at 100.33 59.69 90)
 			(effects
@@
 			)
 		)
-		(property "Value" "1k"
+		(property "Value" "220"
 			(at 100.33 123.19 90)
 			(effects
@@
 			)
 		)
-		(property "Value" "1k"
+		(property "Value" "220"
 			(at 163.83 85.09 90)
 			(effects
