File: 2024-2025_Boards/Spectrometer_Board/Spectrometer V1.0.kicad_pcb (KiCad board)
At the start: 2 copper layers, 56 x 58 mm, 59 parts, among them J1 Conn_01x02_Pin, J2 Conn_01x02_Pin, J3 Conn_ARM_JTAG_SWD_10, J4 Conn_01x03_Socket, J5 Conn_01x03_Socket, J6 Conn_01x04_Socket, J7 Conn_01x02_Pin, U1 LM358N/NOPB, U2 STM32G431CBT6, U3 TCAN1057AEV-Q1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

Commit message: fix
Parts:
- added G***: LOGO, CMR_Logo:CMR_Logo, F.Cu at (121.8, 131.6)
Connections:
- J3 pad 2: /SWCLK -> /SWDIO
- J3 pad 4: /SWDIO -> /SWCLK
Routing:
- net /SWCLK: track 7.91 -> 5.70 mm
- net /SWDIO: track 4.74 -> 6.02 mm
Other:
- board text removed: "David Bascom 2025 V1.0"
Changed lines of the file:
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@@
 			(layers "*.Cu" "*.Mask")
 			(remove_unused_layers no)
-			(net 15 "/SWCLK")
+			(net 17 "/SWDIO")
 			(pinfunction "SWDIO/TMS")
 			(pintype "bidirectional")
@@
 			(layers "*.Cu" "*.Mask")
 			(remove_unused_layers no)
-			(net 17 "/SWDIO")
+			(net 15 "/SWCLK")
 			(pinfunction "SWCLK/TCK")
 			(pintype "output")
@@
 		)
 	)
+	(footprint "CMR_Logo:CMR_Logo"
+		(layer "F.Cu")
+		(at 121.780195 131.555537)
+		(property "Reference" "G***"
+			(at 0 0 -0)
+			(layer "B.SilkS")
+			(hide yes)
+			(effects
+				(font
+					(size 1.5 1.5)
+					(thickness 0.3)
+				)
+				(justify mirror)
+			)
+		)
+		(property "Value" "LOGO"
+			(at -0.75 0 -0)
+			(layer "B.SilkS")
+			(hide yes)
+			(effects
+				(font
+					(size 1.5 1.5)
+					(thickness 0.3)
+				)
+				(justify mirror)
+			)
+		)
+		(property "Footprint" "CMR_Logo:CMR_Logo"
+			(at 0 0 -0)
+			(layer "B.Fab")
+			(hide yes)
+			(effects
+				(font
+					(size 1.27 1.27)
+					(thickness 0.15)
+				)
+				(justify mirror)
+			)
+		)
+		(property "Datasheet" ""
+			(at 0 0 -0)
+			(layer "B.Fab")
+			(hide yes)
+			(effects
+				(font
+					(size 1.27 1.27)
+					(thickness 0.15)
+				)
+				(justify mirror)
+			)
+		)
+		(property "Description" ""
+			(at 0 0 -0)
+			(layer "B.Fab")
+			(hide yes)
+			(effects
+				(font
+					(size 1.27 1.27)
+					(thickness 0.15)
+				)
+				(justify mirror)
+			)
+		)
+		(attr board_only exclude_from_pos_files exclude_from_bom)
+		(fp_poly
+			(pts
+				(xy 0.366889 -2.427111) (xy 0.378511 -2.376777) (xy 0.423333 -2.370666) (xy 0.493023 -2.401645)
+				(xy 0.479778 -2.427111) (xy 0.379298 -2.437244)
+			)
+			(stroke
+				(width 0)
+				(type solid)
+			)
+			(fill solid)
+			(layer "B.SilkS")
+		)
+		(fp_poly
+			(pts
+				(xy 3.045666 -2.854553) (xy 2.963567 -2.785914) (xy 2.963333 -2.780819) (xy 3.04138 -2.682856) (xy 3.251319 -2.58622)
+				(xy 3.355078 -2.555011) (xy 3.765118 -2.377947) (xy 4.05373 -2.112457) (xy 4.208294 -1.782748) (xy 4.216187 -1.413025)
+				(xy 4.109852 -1.107472) (xy 3.853809 -0.754944) (xy 3.465611 -0.401916) (xy 2.980744 -0.071781)
+				(xy 2.434693 0.212067) (xy 1.862942 0.426236) (xy 1.72457 0.465) (xy 1.367542 0.531714) (xy 0.936467 0.573659)
+				(xy 0.484408 0.589773) (xy 0.064428 0.578992) (xy -0.270408 0.540253) (xy -0.396655 0.507506) (xy -0.552619 0.455734)
+				(xy -0.565024 0.472557) (xy -0.469578 0.550625) (xy -0.275605 0.669192) (xy -0.024769 0.757661)
+				(xy 0.308885 0.820419) (xy 0.751313 0.861858) (xy 1.328472 0.886365) (xy 1.545166 0.891335) (xy 2.063115 0.897549)
+				(xy 2.42924 0.892155) (xy 2.660721 0.874092) (xy 2.774738 0.842297) (xy 2.794 0.814058) (xy 2.866274 0.736614)
+				(xy 3.059787 0.614639) (xy 3.339575 0.468983) (xy 3.4925 0.397567) (xy 4.110502 0.070469) (xy 4.607386 -0.291456)
+				(xy 4.978596 -0.674899) (xy 5.219579 -1.066555) (xy 5.325778 -1.453115) (xy 5.292639 -1.821274)
+				(xy 5.115607 -2.157723) (xy 4.790127 -2.449156) (xy 4.518059 -2.598538) (xy 4.208783 -2.71477) (xy 3.868868 -2.802948)
+				(xy 3.536353 -2.85861) (xy 3.249273 -2.877299)
+			)
+			(stroke
+				(width 0)
+				(type solid)
+			)
+			(fill solid)
+			(layer "B.SilkS")
+		)
+		(fp_poly
+			(pts
+				(xy 2.105572 -3.083352) (xy 1.910457 -2.976847) (xy 1.74036 -2.876143) (xy 1.465615 -2.76444) (xy 1.160461 -2.670109)
+				(xy 0.839297 -2.578051) (xy 0.665298 -2.512632) (xy 0.641848 -2.48016) (xy 0.772329 -2.486943) (xy 1.060128 -2.539288)
+				(xy 1.094154 -2.546513) (xy 1.345957 -2.593907) (xy 1.520209 -2.6143) (xy 1.567447 -2.609442) (xy 1.531209 -2.536212)
+				(xy 1.408949 -2.370612) (xy 1.228578 -2.14554) (xy 1.018007 -1.893898) (xy 0.805148 -1.648585) (xy 0.617913 -1.442501)
+				(xy 0.484214 -1.308546) (xy 0.435531 -1.275228) (xy 0.364971 -1.339004) (xy 0.208442 -1.510611)
+				(xy -0.013308 -1.766411) (xy -0.279526 -2.082765) (xy -0.381 -2.205401) (xy -1.143 -3.130345) (xy -3.033346 -3.131506)
+				(xy -4.923692 -3.132666) (xy -5.17118 -2.885179) (xy -5.284229 -2.764282) (xy -5.356264 -2.647777)
+				(xy -5.396513 -2.49505) (xy -5.414207 -2.265483) (xy -5.418575 -1.918462) (xy -5.418667 -1.796058)
+				(xy -5.415899 -1.407242) (xy -5.402008 -1.147765) (xy -5.368616 -0.977655) (xy -5.307344 -0.856941)
+				(xy -5.209813 -0.745652) (xy -5.195455 -0.731212) (xy -4.947666 -0.557537) (xy -4.645121 -0.508)
+				(xy -4.437276 -0.494946) (xy -4.324636 -0.46247) (xy -4.318 -0.451068) (xy -4.369283 -0.364274)
+				(xy -4.505409 -0.18461) (xy -4.699795 0.053286) (xy -4.756621 0.120432) (xy -4.98192 0.384951) (xy -5.177643 0.615122)
+				(xy -5.306899 0.767551) (xy -5.320077 0.783167) (xy -5.381776 0.873015) (xy -5.347534 0.916581)
+				(xy -5.18787 0.930406) (xy -5.055954 0.931334) (xy -4.88292 0.926683) (xy -4.747091 0.897801) (xy -4.617291 0.82229)
+				(xy -4.462343 0.677751) (xy -4.25107 0.441787) (xy -4.054203 0.211667) (xy -3.441408 -0.508) (xy -2.652037 -0.508)
+				(xy -1.862667 -0.508) (xy -1.862667 0.202404) (xy -1.862667 0.912807) (xy -1.568066 0.9472) (xy -1.273465 0.981593)
+				(xy -1.250566 -0.646056) (xy -1.237118 -1.601898) (xy -1.873034 -1.601898) (xy -1.880082 -1.349702)
+				(xy -1.898972 -1.212844) (xy -1.946952 -1.16912) (xy -2.066265 -1.138911) (xy -2.278619 -1.120838)
+				(xy -2.605719 -1.113523) (xy -3.069274 -1.115585) (xy -3.363632 -1.119778) (xy -4.783667 -1.143)
+				(xy -4.783667 -1.820333) (xy -4.783667 -2.497666) (xy -3.344334 -2.497666) (xy -1.905 -2.497666)
+				(xy -1.879674 -1.9134) (xy -1.873034 -1.601898) (xy -1.237118 -1.601898) (xy -1.227667 -2.273705)
+				(xy -0.423334 -1.310622) (xy -0.137101 -0.97213) (xy 0.112366 -0.685082) (xy 0.304586 -0.472429)
+				(xy 0.419081 -0.357127) (xy 0.439936 -0.343103) (xy 0.512183 -0.402898) (xy 0.672335 -0.57065) (xy 0.900115 -0.824042)
+				(xy 1.175246 -1.14076) (xy 1.328936 -1.321462) (xy 2.159 -2.304258) (xy 2.182416 -1.069905) (xy 2.205832 0.164449)
+				(xy 2.499916 0.02421) (xy 2.794 -0.116029) (xy 2.794 -1.624348) (xy 2.794 -3.132666) (xy 2.439623 -3.132666)
+			)
+			(stroke
+				(width 0)
+				(type solid)
+			)
+			(fill solid)
+			(layer "B.SilkS")
+		)
+	)
 	(footprint "LED_SMD:LED_0603_1608Metric"
 		(layer "F.Cu")
@@
 		)
 	)
-	(gr_text "David Bascom\n2025 V1.0"
-		(at 135.8 132.8 0)
-		(layer "B.SilkS")
-		(effects
-			(font
-				(size 2 2)
-				(thickness 0.5)
-				(bold yes)
-			)
-			(justify left bottom mirror)
-		)
-	)
 	(gr_text "BOOT0"
 		(at 140.6 127.4 0)
@@
 	(segment
 		(start 135.87 123.8)
-		(end 137.87 125.8)
+		(end 137.87 121.8)
 		(width 0.3)
 		(layer "F.Cu")
@@
 	)
 	(segment
-		(start 133.055 127.49688)
-		(end 133.055 128.095)
+		(start 137.33 131.08)
+		(end 137.33 131)
 		(width 0.3)
 		(layer "F.Cu")
@@
 	)
 	(segment
-		(start 133.055 128.095)
-		(end 137.31 132.35)
+		(start 135.5 129.25)
+		(end 137.33 131.08)
 		(width 0.3)
 		(layer "F.Cu")
@@
 	)
 	(segment
-		(start 137.33 132.35)
-		(end 137.33 132.27)
+		(start 134.91241 127.25)
+		(end 135.5 127.83759)
 		(width 0.3)
 		(layer "F.Cu")
@@
 	)
 	(segment
-		(start 133.30188 127.25)
-		(end 133.055 127.49688)
+		(start 137.31 131.08)
+		(end 137.33 131.08)
 		(width 0.3)
 		(layer "F.Cu")
@@
 	)
 	(segment
-		(start 134.1425 127.25)
-		(end 133.30188 127.25)
+		(start 135.5 127.83759)
+		(end 135.5 129.25)
 		(width 0.3)
 		(layer "F.Cu")
@@
 	)
 	(segment
-		(start 137.31 132.35)
-		(end 137.33 132.35)
+		(start 134.1425 127.25)
+		(end 134.91241 127.25)
 		(width 0.3)
 		(layer "F.Cu")
@@
 	)
 	(segment
-		(start 135.5 127.98)
-		(end 135.5 126.76688)
+		(start 136 126.5)
+		(end 136 128.48)
 		(width 0.3)
 		(layer "F.Cu")
@@
 	)
 	(segment
-		(start 135.5 126.76688)
-		(end 134.98312 126.25)
+		(start 136 128.48)
+		(end 137.33 129.81)
 		(width 0.3)
 		(layer "F.Cu")
@@
 	)
 	(segment
-		(start 134.98312 126.25)
+		(start 135.75 126.25)
 		(end 134.1425 126.25)
 		(width 0.3)
@@
 	)
 	(segment
-		(start 137.33 129.81)
-		(end 135.5 127.98)
+		(start 136 126.5)
+		(end 135.75 126.25)
 		(width 0.3)
 		(layer "F.Cu")
@@
 	)
 	(segment
-		(start 137.33 131.08)
-		(end 137.33 131)
+		(start 137.33 132.35)
+		(end 137.33 132.27)
 		(width 0.3)
 		(layer "F.Cu")
@@
 	)
 	(segment
-		(start 134.1425 127.75)
-		(end 134.1425 127.9125)
+		(start 134.1425 129.1625)
+		(end 137.33 132.35)
 		(width 0.3)
 		(layer "F.Cu")
@@
 	)
 	(segment
-		(start 137.31 131.08)
-		(end 137.33 131.08)
+		(start 134.1425 127.75)
+		(end 134.1425 129.1625)
 		(width 0.3)
 		(layer "F.Cu")
@@
 	)
 	(segment
-		(start 134.1425 127.9125)
-		(end 137.31 131.08)
+		(start 137.31 132.35)
+		(end 137.33 132.35)
 		(width 0.3)
 		(layer "F.Cu")
