File: 2024-2025_Boards/Spectrometer_Board/Spectrometer V1.0.kicad_sch (KiCad schematic)
At the start: 59 parts, among them J1 Conn_01x02_Pin, J2 Conn_01x02_Pin, J3 Conn_ARM_JTAG_SWD_10, J4 Conn_01x03_Socket, J5 Conn_01x03_Socket, J6 Conn_01x04_Socket, J7 Conn_01x02_Pin, U1 LM358N/NOPB, U2 STM32G431CBT6, U3 TCAN1057AEV-Q1, U4 TL2575-05IKTTR, U5 AMS1117-3.3

Commit message: fix
Connections:
- net SWCLK: now also J3.4 (SWCLK/TCK); no longer J3.2 (SWDIO/TMS)
- net SWDIO: now also J3.2 (SWDIO/TMS); no longer J3.4 (SWCLK/TCK)
Changed lines of the file:
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@@
+	(wire
+		(pts
+			(xy 129.54 95.25) (xy 166.37 95.25)
+		)
+		(stroke
+			(width 0)
+			(type default)
+		)
+	)
 	(wire
 		(pts
@@
 	(wire
 		(pts
+			(xy 129.54 92.71) (xy 168.91 92.71)
+		)
+		(stroke
+			(width 0)
+			(type default)
+		)
+	)
+	(wire
+		(pts
 			(xy 49.53 105.41) (xy 45.72 105.41)
 		)
@@
 	(wire
 		(pts
+			(xy 166.37 119.38) (xy 166.37 95.25)
+		)
+		(stroke
+			(width 0)
+			(type default)
+		)
+	)
+	(wire
+		(pts
 			(xy 134.62 173.99) (xy 134.62 163.83)
 		)
@@
 	(wire
 		(pts
-			(xy 166.37 119.38) (xy 166.37 92.71)
-		)
-		(stroke
-			(width 0)
-			(type default)
-		)
-	)
-	(wire
-		(pts
 			(xy 77.47 116.84) (xy 77.47 115.57)
 		)
@@
 	(wire
 		(pts
+			(xy 168.91 92.71) (xy 168.91 121.92)
+		)
+		(stroke
+			(width 0)
+			(type default)
+		)
+	)
+	(wire
+		(pts
 			(xy 228.6 49.53) (xy 232.41 49.53)
 		)
@@
 	(wire
 		(pts
-			(xy 168.91 95.25) (xy 129.54 95.25)
-		)
-		(stroke
-			(width 0)
-			(type default)
-		)
-	)
-	(wire
-		(pts
 			(xy 191.77 36.83) (xy 191.77 34.29)
 		)
@@
 	(wire
 		(pts
-			(xy 129.54 92.71) (xy 166.37 92.71)
-		)
-		(stroke
-			(width 0)
-			(type default)
-		)
-	)
-	(wire
-		(pts
 			(xy 35.56 49.53) (xy 35.56 48.26)
 		)
@@
 		)
 		(stroke
-			(width 0)
-			(type default)
-		)
-	)
-	(wire
-		(pts
-			(xy 168.91 121.92) (xy 168.91 95.25)
-		)
-		(stroke
