File: 2025-2026_Boards/Fan_Board/Fan_Board/Temp_Sense.kicad_sch (KiCad schematic)
At the start: 1 part, among them U4 TMP275AIDGKR

Commit message: continued layout
Connections:
- net SCL1 renamed SCL2
- net SDA1 renamed SDA2
Changed lines of the file:
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@@
 		)
 	)
-	(global_label "SCL1"
+	(global_label "SCL2"
 		(shape input)
 		(at 114.3 91.44 180)
@@
 		)
 	)
-	(global_label "SDA1"
+	(global_label "SDA2"
 		(shape input)
 		(at 114.3 96.52 180)
