File: 2025-2026_Boards/Stepper_Board/Power.kicad_sch (KiCad schematic)
At the start: 29 parts, among them U1 LM63460AASQRYFRQ1, U2 TLVM23625RDNR, U3 AMS1117-3.3

Commit message: finished driver
Parts:
- added J2, J4: Conn_01x02_Socket, Connector_AMASS:AMASS_XT30PW-M_1x02_P2.50mm_Horizontal, symbol Connector:Conn_01x02_Socket
Connections:
- net +BATT: now also J2.2 (Pin_2), J4.2 (Pin_2)
- net GND: now also J2.1 (Pin_1), J4.1 (Pin_1)
