File: 2025-2026_Boards/Stepper_Board/FDCAN.kicad_sch (KiCad schematic)
At the start: 5 parts, among them J11 Conn_01x03_Socket, J12 Conn_01x03_Socket, U3 TCAN1057AEV-Q1

Commit message: add stuff
Parts:
- renumbered C14 to C31, C15 to C32, J11 to J6, J12 to J7, U3 to U6
Changed lines of the file:
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@@
 		(dnp no)
 		(fields_autoplaced yes)
-		(property "Reference" "U3"
+		(property "Reference" "U6"
 			(at 128.27 71.12 0)
 			(effects
@@
 		(instances
 			(project "Stepper_Board"
-				(path "/afdf0c53-d87b-4ae5-aa44-610ba3220cb0/f1c777ac-0ce7-4e64-94e9-03bc56f74420"
-					(reference "U3")
+				(path "/afdf0c53-d87b-4ae5-aa44-610ba3220cb0/766c7b43-69c9-4b2f-8aa4-0ca55d78a341"
+					(reference "U6")
 					(unit 1)
 				)
@@
 		(on_board yes)
 		(dnp no)
-		(property "Reference" "C14"
+		(property "Reference" "C31"
 			(at 75.692 90.17 0)
 			(effects
@@
 		(instances
 			(project "Stepper_Board"
-				(path "/afdf0c53-d87b-4ae5-aa44-610ba3220cb0/f1c777ac-0ce7-4e64-94e9-03bc56f74420"
-					(reference "C14")
+				(path "/afdf0c53-d87b-4ae5-aa44-610ba3220cb0/766c7b43-69c9-4b2f-8aa4-0ca55d78a341"
+					(reference "C31")
 					(unit 1)
 				)
@@
 		(dnp no)
 		(fields_autoplaced yes)
-		(property "Reference" "J11"
+		(property "Reference" "J6"
 			(at 195.58 82.5499 0)
 			(effects
@@
 		(instances
 			(project "Stepper_Board"
-				(path "/afdf0c53-d87b-4ae5-aa44-610ba3220cb0/f1c777ac-0ce7-4e64-94e9-03bc56f74420"
-					(reference "J11")
+				(path "/afdf0c53-d87b-4ae5-aa44-610ba3220cb0/766c7b43-69c9-4b2f-8aa4-0ca55d78a341"
+					(reference "J6")
 					(unit 1)
 				)
@@
 		(dnp no)
 		(fields_autoplaced yes)
-		(property "Reference" "J12"
+		(property "Reference" "J7"
 			(at 195.58 92.7099 0)
 			(effects
@@
 		(instances
 			(project "Stepper_Board"
-				(path "/afdf0c53-d87b-4ae5-aa44-610ba3220cb0/f1c777ac-0ce7-4e64-94e9-03bc56f74420"
-					(reference "J12")
+				(path "/afdf0c53-d87b-4ae5-aa44-610ba3220cb0/766c7b43-69c9-4b2f-8aa4-0ca55d78a341"
+					(reference "J7")
 					(unit 1)
 				)
@@
 		(instances
 			(project "Stepper_Board"
-				(path "/afdf0c53-d87b-4ae5-aa44-610ba3220cb0/f1c777ac-0ce7-4e64-94e9-03bc56f74420"
+				(path "/afdf0c53-d87b-4ae5-aa44-610ba3220cb0/766c7b43-69c9-4b2f-8aa4-0ca55d78a341"
 					(reference "#PWR037")
 					(unit 1)
@@
 		(instances
 			(project "Stepper_Board"
-				(path "/afdf0c53-d87b-4ae5-aa44-610ba3220cb0/f1c777ac-0ce7-4e64-94e9-03bc56f74420"
+				(path "/afdf0c53-d87b-4ae5-aa44-610ba3220cb0/766c7b43-69c9-4b2f-8aa4-0ca55d78a341"
 					(reference "#PWR034")
 					(unit 1)
@@
 		(instances
 			(project "Stepper_Board"
-				(path "/afdf0c53-d87b-4ae5-aa44-610ba3220cb0/f1c777ac-0ce7-4e64-94e9-03bc56f74420"
+				(path "/afdf0c53-d87b-4ae5-aa44-610ba3220cb0/766c7b43-69c9-4b2f-8aa4-0ca55d78a341"
 					(reference "#PWR036")
 					(unit 1)
@@
 		(instances
 			(project ""
-				(path "/afdf0c53-d87b-4ae5-aa44-610ba3220cb0/f1c777ac-0ce7-4e64-94e9-03bc56f74420"
+				(path "/afdf0c53-d87b-4ae5-aa44-610ba3220cb0/766c7b43-69c9-4b2f-8aa4-0ca55d78a341"
 					(reference "#PWR035")
 					(unit 1)
@@
 		(instances
 			(project ""
-				(path "/afdf0c53-d87b-4ae5-aa44-610ba3220cb0/f1c777ac-0ce7-4e64-94e9-03bc56f74420"
+				(path "/afdf0c53-d87b-4ae5-aa44-610ba3220cb0/766c7b43-69c9-4b2f-8aa4-0ca55d78a341"
 					(reference "#PWR041")
 					(unit 1)
@@
 		(on_board yes)
 		(dnp no)
-		(property "Reference" "C15"
+		(property "Reference" "C32"
 			(at 85.598 90.17 0)
 			(effects
@@
 		(instances
 			(project "Stepper_Board"
-				(path "/afdf0c53-d87b-4ae5-aa44-610ba3220cb0/f1c777ac-0ce7-4e64-94e9-03bc56f74420"
-					(reference "C15")
-					(unit 1)
-				)
+				(path "/afdf0c53-d87b-4ae5-aa44-610ba3220cb0/766c7b43-69c9-4b2f-8aa4-0ca55d78a341"
+					(reference "C32")
+					(unit 1)
+				)
