File: 2025-2026_Boards/Stepper_Board/Stepper_Board.kicad_sch (KiCad schematic)
At the start: 0 parts

Commit message: found driver
Other:
- added sheet Driver (driver.kicad_sch)
Changed lines of the file:
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@@
+		)
+	)
+	(sheet
+		(at 71.12 13.97)
+		(size 49.53 71.12)
+		(exclude_from_sim no)
+		(in_bom yes)
+		(on_board yes)
+		(dnp no)
+		(fields_autoplaced yes)
+		(stroke
+			(width 0.1524)
+			(type solid)
+		)
+		(fill
+			(color 0 0 0 0.0000)
+		)
+		(property "Sheetname" "Driver"
+			(at 71.12 13.2584 0)
+			(effects
+				(font
+					(size 1.27 1.27)
+				)
+				(justify left bottom)
+			)
+		)
+		(property "Sheetfile" "driver.kicad_sch"
+			(at 71.12 85.6746 0)
+			(effects
+				(font
+					(size 1.27 1.27)
+				)
+				(justify left top)
+			)
+		)
+		(instances
+			(project "Stepper_Board"
+				(path "/afdf0c53-d87b-4ae5-aa44-610ba3220cb0"
+					(page "3")
+				)
+			)
 		)
 	)

Commit message: finished driver
Other:
- added sheet MCU (mcu.kicad_sch)
Changed lines of the file:
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@@
 	(paper "A4")
+	(sheet
+		(at 124.46 13.97)
+		(size 50.8 71.12)
+		(exclude_from_sim no)
+		(in_bom yes)
+		(on_board yes)
+		(dnp no)
+		(fields_autoplaced yes)
+		(stroke
+			(width 0.1524)
+			(type solid)
+		)
+		(fill
+			(color 0 0 0 0.0000)
+		)
+		(property "Sheetname" "MCU"
+			(at 124.46 13.2584 0)
+			(effects
+				(font
+					(size 1.27 1.27)
+				)
+				(justify left bottom)
+			)
+		)
+		(property "Sheetfile" "mcu.kicad_sch"
+			(at 124.46 85.6746 0)
+			(effects
+				(font
+					(size 1.27 1.27)
+				)
+				(justify left top)
+			)
+		)
+		(instances
+			(project "Stepper_Board"
+				(path "/afdf0c53-d87b-4ae5-aa44-610ba3220cb0"
+					(page "4")
+				)
+			)
+		)
+	)
 	(sheet
 		(at 13.97 13.97)

Commit message: add stuff
Other:
- added sheet FDCAN (FDCAN.kicad_sch)
- added sheet Test Points (Test_Points.kicad_sch)
Changed lines of the file:
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@@
+	)
+	(sheet
+		(at 236.22 13.97)
+		(size 44.45 71.12)
+		(exclude_from_sim no)
+		(in_bom yes)
+		(on_board yes)
+		(dnp no)
+		(fields_autoplaced yes)
+		(stroke
+			(width 0.1524)
+			(type solid)
+		)
+		(fill
+			(color 0 0 0 0.0000)
+		)
+		(property "Sheetname" "Test Points"
+			(at 236.22 13.2584 0)
+			(effects
+				(font
+					(size 1.27 1.27)
+				)
+				(justify left bottom)
+			)
+		)
+		(property "Sheetfile" "Test_Points.kicad_sch"
+			(at 236.22 85.6746 0)
+			(effects
+				(font
+					(size 1.27 1.27)
+				)
+				(justify left top)
+			)
+		)
+		(instances
+			(project "Stepper_Board"
+				(path "/afdf0c53-d87b-4ae5-aa44-610ba3220cb0"
+					(page "6")
+				)
+			)
+		)
 	)
 	(sheet
@@
 				)
 			)
+		)
+	)
+	(sheet
+		(at 180.34 13.97)
+		(size 49.53 71.12)
+		(exclude_from_sim no)
+		(in_bom yes)
+		(on_board yes)
+		(dnp no)
+		(fields_autoplaced yes)
+		(stroke
+			(width 0.1524)
+			(type solid)
+		)
+		(fill
+			(color 0 0 0 0.0000)
+		)
+		(property "Sheetname" "FDCAN"
+			(at 180.34 13.2584 0)
+			(effects
+				(font
+					(size 1.27 1.27)
+				)
+				(justify left bottom)
+			)
+		)
+		(property "Sheetfile" "FDCAN.kicad_sch"
+			(at 180.34 85.6746 0)
+			(effects
+				(font
+					(size 1.27 1.27)
+				)
+				(justify left top)
+			)
+		)
+		(instances
+			(project "Stepper_Board"
+				(path "/afdf0c53-d87b-4ae5-aa44-610ba3220cb0"
+					(page "5")
+				)
+			)
