File: 2025-2026_Boards/Stepper_Board/mcu.kicad_sch (KiCad schematic)
At the start: 18 parts, among them J1 Conn_01x02_Pin, J3 Conn_ARM_JTAG_SWD_10, U5 STM32G431CBT6

Commit message: add stuff
Parts:
- renumbered D18 to D4, D17 to D5, R30 to R12, R29 to R13
Connections:
- net MISO: now also U5.14 (PA6); no longer U5.43 (PB6)
- net MOSI: now also U5.15 (PA7); no longer U5.44 (PB7)
- net SCLK: now also U5.13 (PA5); no longer U5.42 (PB5)
- net DIR: now reaches U5.10 (PA2)
- net STEP: now reaches U5.11 (PA3)
- net CS: now reaches U5.12 (PA4)
- net nSLEEP: now reaches U5.8 (PA0)
- net Enable: now reaches U5.9 (PA1)
Changed lines of the file:
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@@
+	(wire
+		(pts
+			(xy 163.83 81.28) (xy 166.37 81.28)
+		)
+		(stroke
+			(width 0)
+			(type default)
+		)
+	)
 	(wire
 		(pts
@@
 	(wire
 		(pts
+			(xy 166.37 83.82) (xy 163.83 83.82)
+		)
+		(stroke
+			(width 0)
+			(type default)
+		)
+	)
+	(wire
+		(pts
 			(xy 166.37 106.68) (xy 166.37 125.73)
 		)
@@
 	(wire
 		(pts
-			(xy 123.19 111.76) (xy 130.81 111.76)
-		)
-		(stroke
-			(width 0)
-			(type default)
-		)
-	)
-	(wire
-		(pts
-			(xy 123.19 116.84) (xy 130.81 116.84)
-		)
-		(stroke
-			(width 0)
-			(type default)
-		)
-	)
-	(wire
-		(pts
 			(xy 195.58 130.81) (xy 198.12 130.81)
 		)
@@
 	(wire
 		(pts
+			(xy 166.37 73.66) (xy 163.83 73.66)
+		)
+		(stroke
+			(width 0)
+			(type default)
+		)
+	)
+	(wire
+		(pts
 			(xy 93.98 76.2) (xy 130.81 76.2)
 		)
@@
 	(wire
 		(pts
+			(xy 163.83 78.74) (xy 166.37 78.74)
+		)
+		(stroke
+			(width 0)
+			(type default)
+		)
+	)
+	(wire
+		(pts
 			(xy 80.01 76.2) (xy 91.44 76.2)
 		)
@@
 	(wire
 		(pts
+			(xy 166.37 86.36) (xy 163.83 86.36)
+		)
+		(stroke
+			(width 0)
+			(type default)
+		)
+	)
+	(wire
+		(pts
 			(xy 129.54 71.12) (xy 130.81 71.12)
 		)
@@
 	(wire
 		(pts
+			(xy 166.37 76.2) (xy 163.83 76.2)
+		)
+		(stroke
+			(width 0)
+			(type default)
+		)
+	)
+	(wire
+		(pts
 			(xy 163.83 50.8) (xy 175.26 50.8)
 		)
@@
 	(wire
 		(pts
+			(xy 166.37 71.12) (xy 163.83 71.12)
+		)
+		(stroke
+			(width 0)
+			(type default)
+		)
+	)
+	(wire
+		(pts
 			(xy 143.51 64.77) (xy 143.51 66.04)
 		)
@@
 	(wire
 		(pts
-			(xy 123.19 114.3) (xy 130.81 114.3)
-		)
-		(stroke
-			(width 0)
-			(type default)
-		)
-	)
-	(wire
-		(pts
 			(xy 81.28 50.8) (xy 69.85 50.8)
 		)
@@
 	(wire
 		(pts
+			(xy 166.37 88.9) (xy 163.83 88.9)
+		)
+		(stroke
+			(width 0)
+			(type default)
+		)
+	)
+	(wire
+		(pts
 			(xy 129.54 64.77) (xy 143.51 64.77)
 		)
@@
 			(width 0)
 			(type default)
+		)
+	)
+	(global_label "STEP"
+		(shape input)
+		(at 166.37 78.74 0)
+		(fields_autoplaced yes)
+		(effects
+			(font
+				(size 1.27 1.27)
+			)
+			(justify left)
+		)
+		(property "Intersheetrefs" "${INTERSHEET_REFS}"
+			(at 173.9513 78.74 0)
+			(effects
+				(font
+					(size 1.27 1.27)
+				)
+				(justify left)
+				(hide yes)
+			)
+		)
+	)
+	(global_label "SCLK"
+		(shape input)
+		(at 166.37 83.82 0)
+		(fields_autoplaced yes)
+		(effects
+			(font
+				(size 1.27 1.27)
+			)
+			(justify left)
+		)
+		(property "Intersheetrefs" "${INTERSHEET_REFS}"
+			(at 174.1328 83.82 0)
+			(effects
+				(font
+					(size 1.27 1.27)
+				)
+				(justify left)
+				(hide yes)
+			)
 		)
 	)
@@
 		)
 	)
+	(global_label "CS"
+		(shape input)
+		(at 166.37 81.28 0)
+		(fields_autoplaced yes)
+		(effects
+			(font
+				(size 1.27 1.27)
+			)
+			(justify left)
+		)
+		(property "Intersheetrefs" "${INTERSHEET_REFS}"
+			(at 171.8347 81.28 0)
+			(effects
+				(font
+					(size 1.27 1.27)
+				)
+				(justify left)
+				(hide yes)
+			)
+		)
+	)
+	(global_label "Enable"
+		(shape input)
+		(at 166.37 73.66 0)
+		(fields_autoplaced yes)
+		(effects
+			(font
+				(size 1.27 1.27)
+			)
+			(justify left)
+		)
+		(property "Intersheetrefs" "${INTERSHEET_REFS}"
+			(at 175.705 73.66 0)
+			(effects
+				(font
+					(size 1.27 1.27)
+				)
+				(justify left)
+				(hide yes)
+			)
+		)
+	)
 	(global_label "NREST"
 		(shape input)
@@
 		)
 	)
-	(global_label "SCLK"
+	(global_label "nSLEEP"
 		(shape input)
-		(at 123.19 111.76 180)
+		(at 166.37 71.12 0)
 		(fields_autoplaced yes)
 		(effects
@@
 				(size 1.27 1.27)
 			)
-			(justify right)
+			(justify left)
 		)
 		(property "Intersheetrefs" "${INTERSHEET_REFS}"
-			(at 115.4272 111.76 0)
-			(effects
-				(font
-					(size 1.27 1.27)
-				)
-				(justify right)
+			(at 176.3098 71.12 0)
+			(effects
+				(font
+					(size 1.27 1.27)
+				)
+				(justify left)
 				(hide yes)
 			)
@@
 		)
 	)
-	(global_label "MISO"
+	(global_label "DIR"
 		(shape input)
-		(at 123.19 114.3 180)
+		(at 166.37 76.2 0)
 		(fields_autoplaced yes)
 		(effects
@@
 				(size 1.27 1.27)
 			)
-			(justify right)
+			(justify left)
 		)
 		(property "Intersheetrefs" "${INTERSHEET_REFS}"
-			(at 115.6086 114.3 0)
-			(effects
-				(font
-					(size 1.27 1.27)
-				)
-				(justify right)
+			(at 172.5 76.2 0)
+			(effects
+				(font
+					(size 1.27 1.27)
+				)
+				(justify left)
+				(hide yes)
+			)
+		)
+	)
+	(global_label "MOSI"
+		(shape input)
+		(at 166.37 88.9 0)
+		(fields_autoplaced yes)
+		(effects
+			(font
+				(size 1.27 1.27)
+			)
+			(justify left)
+		)
+		(property "Intersheetrefs" "${INTERSHEET_REFS}"
+			(at 173.9514 88.9 0)
+			(effects
+				(font
+					(size 1.27 1.27)
+				)
+				(justify left)
 				(hide yes)
 			)
@@
 		)
 	)
-	(global_label "MOSI"
+	(global_label "NREST"
 		(shape input)
-		(at 123.19 116.84 180)
+		(at 195.58 120.65 180)
 		(fields_autoplaced yes)
 		(effects
@@
 		)
 		(property "Intersheetrefs" "${INTERSHEET_REFS}"
-			(at 115.6086 116.84 0)
+			(at 186.6682 120.65 0)
 			(effects
 				(font
@@
 		)
 	)
-	(global_label "NREST"
+	(global_label "MISO"
 		(shape input)
-		(at 195.58 120.65 180)
+		(at 166.37 86.36 0)
 		(fields_autoplaced yes)
 		(effects
@@
 				(size 1.27 1.27)
 			)
-			(justify right)
+			(justify left)
 		)
 		(property "Intersheetrefs" "${INTERSHEET_REFS}"
-			(at 186.6682 120.65 0)
-			(effects
-				(font
-					(size 1.27 1.27)
-				)
-				(justify right)
+			(at 173.9514 86.36 0)
+			(effects
+				(font
+					(size 1.27 1.27)
+				)
+				(justify left)
 				(hide yes)
 			)
@@
 		(dnp no)
 		(fields_autoplaced yes)
-		(property "Reference" "D17"
+		(property "Reference" "D5"
 			(at 106.3625 85.09 0)
 			(effects
@@
 			(project "Stepper_Board"
 				(path "/afdf0c53-d87b-4ae5-aa44-610ba3220cb0/03775ae2-2f8b-4b47-a8b3-c4248829d87d"
-					(reference "D17")
+					(reference "D5")
 					(unit 1)
 				)
@@
 		(dnp no)
 		(fields_autoplaced yes)
-		(property "Reference" "R29"
+		(property "Reference" "R13"
 			(at 97.79 85.09 90)
 			(effects
@@
 			(project "Stepper_Board"
 				(path "/afdf0c53-d87b-4ae5-aa44-610ba3220cb0/03775ae2-2f8b-4b47-a8b3-c4248829d87d"
-					(reference "R29")
+					(reference "R13")
 					(unit 1)
 				)
@@
 		(dnp no)
 		(fields_autoplaced yes)
-		(property "Reference" "R30"
+		(property "Reference" "R12"
 			(at 78.74 87.63 90)
 			(effects
@@
 			(project "Stepper_Board"
 				(path "/afdf0c53-d87b-4ae5-aa44-610ba3220cb0/03775ae2-2f8b-4b47-a8b3-c4248829d87d"
-					(reference "R30")
+					(reference "R12")
 					(unit 1)
 				)
@@
 		(dnp no)
 		(fields_autoplaced yes)
-		(property "Reference" "D18"
+		(property "Reference" "D4"
 			(at 87.3125 87.63 0)
 			(effects
@@
 			(project "Stepper_Board"
 				(path "/afdf0c53-d87b-4ae5-aa44-610ba3220cb0/03775ae2-2f8b-4b47-a8b3-c4248829d87d"
-					(reference "D18")
+					(reference "D4")
 					(unit 1)
 				)
