File: 2025-2026_Boards/Fan_Board/mcu.kicad_sch (KiCad schematic)
At the start: 25 parts, among them J1 Conn_01x02_Pin, J2 Conn_ARM_JTAG_SWD_10, J21 Conn_01x02_Pin, U3 STM32G431CBT6

Commit message: added labels
Connections:
- no-connect marks 24 -> 25
Changed lines of the file:
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@@
+	)
+	(no_connect
+		(at 162.56 78.74)
 	)
 	(no_connect
