File: 2024-2025_Boards/BDC_Board/CAN.kicad_sch (KiCad schematic)
At the start: 5 parts, among them J4 Conn_01x03_Socket, J5 Conn_01x03_Socket, U6 TCAN1057AEV-Q1

Commit message: add stuff
Changed lines of the file:
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@@
 (kicad_sch
-	(version 20231120)
+	(version 20250114)
 	(generator "eeschema")
-	(generator_version "8.0")
+	(generator_version "9.0")
 	(paper "A4")
 	(junction
