File: 2024-2025_Boards/BDC_Board/Motor_Ports.kicad_sch (KiCad schematic)
At the start: 30 parts, among them J10 Conn_01x02_Socket, J11 Conn_01x02_Socket, J12 Conn_01x02_Socket, J13 Conn_01x02_Socket, J8 Conn_01x02_Socket, J9 Conn_01x02_Socket

Commit message: add stuff
Changed lines of the file:
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@@
 (kicad_sch
-	(version 20231120)
+	(version 20250114)
 	(generator "eeschema")
-	(generator_version "8.0")
+	(generator_version "9.0")
 	(paper "A4")
 	(junction
