File: 2024-2025_Boards/BDC_Board/Power.kicad_sch (KiCad schematic)
At the start: 33 parts, among them J18 Conn_02x10_Odd_Even, J6 Conn_01x02_Socket, J7 Conn_01x02_Socket, Q1 DMPH6023SK3-13, U4 NCP1117ST50T3G, U5 AMS1117-3.3

Commit message: add stuff
Connections:
- net +5V: no longer D2.1 (K), R9.1
- new net: D2.1 (K), R9.1
Changed lines of the file:
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@@
 (kicad_sch
-	(version 20231120)
+	(version 20250114)
 	(generator "eeschema")
-	(generator_version "8.0")
+	(generator_version "9.0")
 	(paper "A4")
 	(junction
@@
 	)
 	(junction
-		(at 143.51 38.1)
-		(diameter 0)
-		(color 0 0 0 0)
-	)
-	(junction
 		(at 182.88 38.1)
 		(diameter 0)
@@
 		)
 		(stroke
-			(width 0)
-			(type default)
-		)
-	)
-	(wire
-		(pts
-			(xy 143.51 38.1) (xy 153.67 38.1)
-		)
-		(stroke
