File: 2024-2025_Boards/BDC_Board/Sensors.kicad_sch (KiCad schematic)
At the start: 12 parts, among them U13 LM35-D, U7 INA2180A1IDGKR, U8 INA2180A1IDGKR, U9 INA2180A1IDGKR

Commit message: add stuff
Changed lines of the file:
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@@
 (kicad_sch
-	(version 20231120)
+	(version 20250114)
 	(generator "eeschema")
-	(generator_version "8.0")
+	(generator_version "9.0")
 	(paper "A4")
 	(junction
