File: 2024-2025_Boards/BDC_Board/V1.0.kicad_pcb (KiCad board)
At the start: 2 copper layers, 88 x 65 mm, 152 parts, among them J1 Conn_01x02_Pin, J10 Conn_01x02_Socket, J11 Conn_01x02_Socket, J12 Conn_01x02_Socket, J13 Conn_01x02_Socket, J14 Conn_01x07_Socket, J15 Conn_01x07_Socket, J16 Conn_01x07_Socket, J18 Conn_02x10_Odd_Even, J2 Conn_01x02_Pin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

Commit message: add stuff
Connections:
- D2 pad 1: +5V -> Net-(D2-K)
- R9 pad 1: +5V -> Net-(D2-K)
Routing:
- net Net-(D2-K): track 0.00 -> 1.89 mm
- net +5V: track 72.5 -> 70.6 mm
Other:
- board size 88 x 65 mm -> 88.5 x 65 mm
