File: 2024-2025_Boards/BDC_Board/V1.0.kicad_sch (KiCad schematic)
At the start: 0 parts

Commit message: auxport no longer name problem
Other:
- sheet AUX renamed AUX_Port
Changed lines of the file:
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@@
 			(color 0 0 0 0.0000)
 		)
-		(property "Sheetname" "AUX"
+		(property "Sheetname" "AUX_Port"
 			(at 162.56 116.1284 0)
 			(effects
